File: sensor.sch (EAGLE design)
At the start: 30 parts, among them IC1 LM339N, IC2 7805TV

Commit message: Transistor und Vorwiderstand
Parts:
- C8: device resistor:C-EU050-025X075 -> resistor:CPOL-EUE3.5-8
- R13: value (none) -> 470R
- T1: value (none) -> BC 141-10
Connections:
- net DIGITAL_OUT: now also C8.+; no longer C8.1
- net GND: now also C8.-; no longer C8.2
Changed lines of the file:
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@@
 <part name="C7" library="resistor" deviceset="C-EU" device="050-025X075" value="5p"/>
 <part name="L1" library="inductors" deviceset="BC12" device="" value="1m"/>
-<part name="C8" library="resistor" deviceset="C-EU" device="050-025X075" value="1u5"/>
 <part name="R9" library="resistor" deviceset="R-EU_" device="0207/7" value="4k7"/>
 <part name="R11" library="resistor" deviceset="R-EU_" device="0207/7" value="2k7"/>
@@
 <part name="GND6" library="supply1" deviceset="GND" device=""/>
 <part name="LED2" library="led" deviceset="LED" device="5MM" value="rt"/>
-<part name="R13" library="resistor" deviceset="R-EU_" device="0207/7"/>
+<part name="R13" library="resistor" deviceset="R-EU_" device="0207/7" value="470R"/>
 <part name="SUPPLY6" library="supply2" deviceset="VDD" device=""/>
 <part name="SUPPLY7" library="supply2" deviceset="VDD" device=""/>
-<part name="T1" library="transistor-neu-to92" deviceset="*-NPN-" device="TO92"/>
+<part name="T1" library="transistor-neu-to92" deviceset="*-NPN-" device="TO92" value="BC 141-10"/>
 <part name="R14" library="resistor" deviceset="R-EU_" device="0207/7" value="270R"/>
+<part name="C8" library="resistor" deviceset="CPOL-EU" device="E3.5-8" value="1u5"/>
 </parts>
 <sheets>
@@
 <instance part="C7" gate="G$1" x="347.98" y="180.34" rot="R180"/>
 <instance part="L1" gate="G$1" x="347.98" y="154.94" rot="R90"/>
-<instance part="C8" gate="G$1" x="215.9" y="83.82"/>
 <instance part="R9" gate="G$1" x="215.9" y="104.14" rot="R90"/>
 <instance part="R11" gate="G$1" x="256.54" y="81.28" rot="R90"/>
@@
 <instance part="T1" gate="G$1" x="40.64" y="111.76"/>
 <instance part="R14" gate="G$1" x="43.18" y="96.52" rot="R270"/>
+<instance part="C8" gate="G$1" x="215.9" y="86.36"/>
 </instances>
 <busses>
@@
 <pinref part="GND4" gate="1" pin="GND"/>
 <wire x1="256.54" y1="76.2" x2="215.9" y2="76.2" width="0.1524" layer="91"/>
-<pinref part="C8" gate="G$1" pin="2"/>
+<pinref part="C8" gate="G$1" pin="-"/>
 <wire x1="215.9" y1="76.2" x2="203.2" y2="76.2" width="0.1524" layer="91"/>
-<wire x1="215.9" y1="78.74" x2="215.9" y2="76.2" width="0.1524" layer="91"/>
+<wire x1="215.9" y1="81.28" x2="215.9" y2="76.2" width="0.1524" layer="91"/>
 <junction x="215.9" y="76.2"/>
 </segment>
@@
 <net name="DIGITAL_OUT" class="0">
 <segment>
-<pinref part="C8" gate="G$1" pin="1"/>
 <pinref part="R9" gate="G$1" pin="1"/>
-<wire x1="215.9" y1="86.36" x2="215.9" y2="93.98" width="0.1524" layer="91"/>
 <pinref part="IC1" gate="A" pin="OUT"/>
 <wire x1="215.9" y1="93.98" x2="215.9" y2="99.06" width="0.1524" layer="91"/>
@@
 <wire x1="215.9" y1="93.98" x2="198.12" y2="93.98" width="0.1524" layer="91"/>
 <label x="180.34" y="93.98" size="1.778" layer="95"/>
-</segment>
-<segment>
+<pinref part="C8" gate="G$1" pin="+"/>
+<wire x1="215.9" y1="88.9" x2="215.9" y2="93.98" width="0.1524" layer="91"/>
+</segment>
+<segment>

Commit message: µC und RS485-Treiber eingefügt
Parts:
- added C10, C11: 12p, resistor:C-EU050-025X075
- added C9: 100n, resistor:C-EU050-025X075
- added IC3: MAX481CPA, maxim:MAX481CPA
- added IC4: ATTINY24/44/84-PU, attiny24_44_84:ATTINY24/44/84-PU
- added Q1: 16MHz, special:XTAL
- added R15: 10k, resistor:R-EU_0207/7
- added U$1: AVR_ISP, n39:AVR_ISP
Connections:
- new net 485_A: IC3G$1.A
- new net 485_B: IC3G$1.B
- new net 485_DE: IC3G$1.DE, IC4.(PCINT3/T0/ADC3)PA3
- new net 485_DI: IC3G$1.DI, IC4.(PCINT2/AIN1/ADC2)PA2
- new net 485_RO: IC3G$1.RO, IC4.(PCINT7/ICP/OC0B/ADC7)PA7
- new net ALARM: IC4.(PCINT10/INT0/OC0A/CKOUT)PB2
- new net MISO: IC4.(PCINT5/OC1B/MISO/DO/ADC5)PA5, U$1.MISO
- new net RST: IC4.(PCINT11/RESET/DW)PB3, R15.1, U$1.RST
- new net SCL: IC4.(PCINT4/T1/SCL/USCK/ADC4)PA4, U$1.SCK
- new net SDA: IC4.(PCINT6/OC1A/SDA/MOSI/ADC6)PA6, U$1.MOSI
- new net XTAL1: C11.1, IC4.(PCINT8/XTAL1/CLKI)PB0, Q1.1
- new net XTAL2: C10.1, IC4.(PCINT9/XTAL2)PB1, Q1.2
- net ANALOG_OUT: now also IC4.(PCINT1/AIN0/ADC1)PA1
- net GND: now also C10.2, C11.2, C9.2, IC3G$1.RE/, IC4.GND
- net HEATER: now also IC4.(PCINT0/AREF/ADC0)PA0
- net VCC: now also C9.1, IC4.VCC, R15.2
